File: Eagle Files/495Group10/gr10-1.brd (EAGLE design)
At the start: 88.6 x 48.2 mm, 51 parts, among them Y1 16MHz, Y2 16 MHZ

Commit message: Fixed a few things in the Main Board.
I updated the main board to use the new Radio part.
I also changed the ground plane distance to 20 mil.

--Arthur

git-svn-id: http://cd-net.net/CPE496/trunk@86 05b6d0e0-c345-4a8e-a5b7-579c8bd0b646
Routing:
- net N$3: track 15.9 -> 12.6 mm
Changed lines of the file:
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@@
 <contactref element="U$4" pad="GNDDC"/>
 <contactref element="U$4" pad="GND"/>
-<polygon width="0.254" layer="16" isolate="1.27" thermals="no">
+<polygon width="0.254" layer="16" isolate="0.508" thermals="no">
 <vertex x="88.9" y="48.26"/>
 <vertex x="0" y="48.26"/>
@@
 <contactref element="MT2201" pad="8"/>
 <contactref element="B1" pad="~2"/>
-<wire x1="39.1668" y1="11.0744" x2="39.1668" y2="2.51" width="1.27" layer="1"/>
-<wire x1="39.1668" y1="2.51" x2="46.48" y2="2.51" width="1.27" layer="1"/>
+<wire x1="39.1668" y1="11.0744" x2="39.1668" y2="8.0644" width="1.27" layer="1"/>
+<wire x1="39.1668" y1="8.0644" x2="44.7212" y2="2.51" width="1.27" layer="1"/>
+<wire x1="44.7212" y1="2.51" x2="46.48" y2="2.51" width="1.27" layer="1"/>
 </signal>
 <signal name="RESET">

Commit message: Updated Boards
--Arthur

git-svn-id: http://cd-net.net/CPE496/trunk@93 05b6d0e0-c345-4a8e-a5b7-579c8bd0b646
Parts:
- moved R2 13.8 mm to (71.1, 30.2), turned to 90 degrees
Routing:
- net MOSI: track 62.3 -> 10.3 mm, vias 4 -> 1
- net MISO: track 72.2 -> 29.7 mm, vias 2 -> 1
- net SCK: track 75.2 -> 42.1 mm
- net CLKM: track 20.5 -> 0.00 mm, vias 2 -> 0
- net 3.3V: track 226.1 -> 210.6 mm
- net CS-RADIO: track 21.0 -> 28.2 mm
- net IRQ: track 8.91 -> 15.5 mm, vias 0 -> 1
- net RADIO-RST: track 34.2 -> 37.8 mm
