File: Eagle Files/Main Board with Headers/Main Board.brd (EAGLE design)
At the start: 67.3 x 43.2 mm, 52 parts, among them IC1 FT232RL, X2 MINI-USB-UX60A-MB-5ST, Y1 16MHz, Y2 16 MHZ

Commit message: Updated the Board we're having made.
--Arthur

git-svn-id: http://cd-net.net/CPE496/trunk@127 05b6d0e0-c345-4a8e-a5b7-579c8bd0b646
Parts:
- removed U$1: MICROSD, group10:MICRO-SD-SOCKET-PP
- removed U$2: ATMEGA32832A, group10:TQFP32-08
- removed U$3: AT86RF231(RADIO)AT86RF231, group10:32QN2(RADIO)
- removed U$4: WE-BAL, group10:WE-BAL
- removed U$5: ANTENNA2SMD, SparkFun:ANTENNA-CHIP2
- added ANTENNA: ANTENNA2SMD, SparkFun:ANTENNA-CHIP2
- added AT86RF231: AT86RF231(RADIO)AT86RF231, group10:32QN2(RADIO)
- added ATMEGA328: ATMEGA32832A, group10:TQFP32-08
- added BALUN: WE-BAL, group10:WE-BAL
- added C12: 10 nF, SparkFun:0603-CAP
- added MICROSD: MICROSD, group10:MICRO-SD-SOCKET-PP
- ACHOT, ACNEU, ACOUT: device wirepad:3,81/1,4 -> group10:PTH-3MM
- C3, C4: value 22p -> 22 pF
- MT2201: value (none) -> 115V -> 5V
- RF-RX: value GREEN -> Green
- RF-TX: value RED -> Red
- Y1: value 16MHz -> 16 MHZ
- moved C3 2.54 mm to (67.3, 9.78)
- moved C4 2.54 mm to (67.3, 18.2)
- moved CX1 2.54 mm to (66.5, 34.3)
- moved CX2 2.54 mm to (66.5, 27.9)
- moved R2 2.54 mm to (44.5, 30.5)
- moved R4 2.54 mm to (44.5, 33.0)
- moved RF-RX 2.54 mm to (53.3, 33.1)
- moved C5 2.54 mm to (26.7, 14.0)
- moved C7 2.54 mm to (26.7, 32.4)
- moved C1 2.54 mm to (16.3, 29.2)
- moved C2 2.54 mm to (17.0, 23.9)
- moved 3.3V_REGULATOR 2.54 mm to (27.8, 4.06)
- moved B1 2.54 mm to (32.1, 14.6)
- moved B2 2.54 mm to (32.4, 28.4)
- moved C10 2.54 mm to (50.2, 33.0)
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Connections:
- removed net RXLED: IC1.22
- removed net TXLED: IC1.23
- new net 3.3V1: 3.3V_REGULATOR.4, C12.2
- net 3.3V: now also AT86RF231.DEVDD, AT86RF231.EVDD, ATMEGA328.18, ATMEGA328.4, ATMEGA328.6, IC1.17, MICROSD.4; no longer U$1.4, U$2.18, U$2.4, U$2.6, U$3.DEVDD, U$3.EVDD
- net CS-RADIO: now also AT86RF231./SEL, ATMEGA328.14; no longer U$2.14, U$3./SEL
- net CS-SD_CARD: now also ATMEGA328.1, MICROSD.2; no longer U$1.2, U$2.1
- net DIG2: now also AT86RF231.DIG2, ATMEGA328.11; no longer U$2.11, U$3.DIG2
- net GND: now also AT86RF231.AVSS, AT86RF231.AVSS2, AT86RF231.AVSS3, AT86RF231.AVSS4, AT86RF231.AVSS5, AT86RF231.AVSS6, AT86RF231.DIG1, AT86RF231.DVSS, AT86RF231.DVSS2, AT86RF231.DVSS3, AT86RF231.DVSS4, AT86RF231.DVSS5, AT86RF231.GND, ATMEGA328.21, ATMEGA328.3, ATMEGA328.5, BALUN.GND, BALUN.GNDDC, C12.1, MICROSD.6; no longer U$1.6, U$2.21, U$2.3, U$2.5, U$3.AVSS, U$3.AVSS2, U$3.AVSS3, U$3.AVSS4, U$3.AVSS5, U$3.AVSS6, U$3.DIG1, U$3.DVSS, U$3.DVSS3, U$3.DVSS4, U$3.DVSS5, U$4.GND, U$4.GNDDC
- net IRQ: now also AT86RF231.IRQ, ATMEGA328.13; no longer U$2.13, U$3.IRQ
- net LED-OUT: now also ATMEGA328.9; no longer U$2.9
- net MISO: now also AT86RF231.MISO, ATMEGA328.16, MICROSD.7; no longer U$1.7, U$2.16, U$3.MISO
- net MOSI: now also AT86RF231.MOSI, ATMEGA328.15, MICROSD.3; no longer U$1.3, U$2.15, U$3.MOSI
- net N$10: now also AT86RF231.AVDD; no longer U$3.AVDD
- net N$11: now also AT86RF231.XTAL1; no longer U$3.XTAL1
- net N$12: now also AT86RF231.XTAL2; no longer U$3.XTAL2
- net N$13: now also AT86RF231.DIG4; no longer U$3.DIG4
- net N$15: now also AT86RF231.DIG3; no longer U$3.DIG3
- net N$16: now also BALUN.OUT2; no longer U$4.OUT2
- net N$17: now also BALUN.OUT1; no longer U$4.OUT1
- net N$18: now also AT86RF231.RFN; no longer U$3.RFN
- net N$19: now also AT86RF231.RFP; no longer U$3.RFP
- net N$20: now also ANTENNA.FEED, BALUN.IN; no longer U$4.IN, U$5.FEED
- net N$8: now also AT86RF231.DVDD, AT86RF231.DVDD2; no longer U$3.DVDD, U$3.DVDD2
- net PC0: now also ATMEGA328.23; no longer U$2.23
- net PC1: now also ATMEGA328.24; no longer U$2.24
- net RADIO-RST: now also AT86RF231./RST, ATMEGA328.10; no longer U$2.10, U$3./RST
- net RESET: now also ATMEGA328.29; no longer U$2.29
- net SCK: now also AT86RF231.SCLK, ATMEGA328.17, MICROSD.5; no longer U$1.5, U$2.17, U$3.SCLK
- net SERIAL-IN: now also ATMEGA328.30; no longer U$2.30
- net SERIAL-OUT: now also ATMEGA328.31; no longer U$2.31
- net SLP_TR: now also AT86RF231.SLP_TR, ATMEGA328.12; no longer U$2.12, U$3.SLP_TR
- net XTAL1: now also ATMEGA328.7; no longer U$2.7
- net XTAL2: now also ATMEGA328.8; no longer U$2.8
Routing:
- net GND: track 122.1 -> 112.5 mm, vias 14 -> 15
- net N$2: track 4.17 -> 10.6 mm
- net N$1: track 10.4 -> 16.1 mm
- net 3.3V1: track 0.00 -> 3.12 mm
- net 3.3V: track 162.5 -> 164.2 mm
- net SERIAL-OUT: track 62.9 -> 63.8 mm
- net SERIAL-IN: track 54.8 -> 55.5 mm
- net N$9: track 6.00 -> 6.65 mm
- net N$8: track 3.77 -> 4.29 mm
- net D-: vias 1 -> 0
Other:
- board size 67.3 x 43.2 mm -> 69.8 x 43.2 mm
- board text added: "CPE 496 Group 10 REV: A"
